Commit message: fix size of small_box

File: hrpsys_gazebo_tutorials/environment_models/small_box/model1.urdf (robot description, URDF)
Before this commit: robot small_box, 15 links, 14 joints
Links:
- link nil_link1: geometry collision box size=0.20 0.315 0.61; visual box size=0.20 0.315 0.61
Joints:
- joint LHAND_DUMMY: origin xyz=0.30 -0.30 0.40 rpy=3.14159 -1.5708 0 -> xyz=0.23 -0.20 0.20 rpy=3.14159 -1.5708 0
- joint RHAND_DUMMY: origin xyz=0.30 0.30 0.40 rpy=3.14159 -1.5708 0 -> xyz=0.23 0.20 0.20 rpy=3.14159 -1.5708 0

File: hrpsys_gazebo_tutorials/environment_models/small_box/model1.urdf.xacro (robot description, xacro)
@@ -8,5 +8,5 @@
   </xacro:include>
   <joint name="LHAND_DUMMY" type="revolute">
-    <origin xyz="0.30 -0.30 0.40" rpy="3.14159 -1.5708 0"/>
+    <origin xyz="0.23 -0.20 0.20" rpy="3.14159 -1.5708 0"/>
     <parent link="nil_link"/>
     <child link="LARM_LINK6"/>
@@ -16,5 +16,5 @@
   </joint>
   <joint name="RHAND_DUMMY" type="revolute">
-    <origin xyz="0.30 0.30 0.40" rpy="3.14159 -1.5708 0"/>
+    <origin xyz="0.23 0.20 0.20" rpy="3.14159 -1.5708 0"/>
     <parent link="nil_link"/>
     <child link="RARM_LINK6"/>

File: hrpsys_gazebo_tutorials/environment_models/small_box/model2.urdf (robot description, URDF)
Before this commit: robot small_box, 15 links, 14 joints
Links:
- link nil_link2: geometry collision box size=0.20 0.315 0.61; visual box size=0.20 0.315 0.61
Joints:
- joint LHAND_DUMMY: origin xyz=0.30 -0.30 0.40 rpy=3.14159 -1.5708 0 -> xyz=0.23 -0.20 0.20 rpy=3.14159 -1.5708 0
- joint RHAND_DUMMY: origin xyz=0.30 0.30 0.40 rpy=3.14159 -1.5708 0 -> xyz=0.23 0.20 0.20 rpy=3.14159 -1.5708 0

File: hrpsys_gazebo_tutorials/environment_models/small_box/model2.urdf.xacro (robot description, xacro)
@@ -8,5 +8,5 @@
   </xacro:include>
   <joint name="LHAND_DUMMY" type="revolute">
-    <origin xyz="0.30 -0.30 0.40" rpy="3.14159 -1.5708 0"/>
+    <origin xyz="0.23 -0.20 0.20" rpy="3.14159 -1.5708 0"/>
     <parent link="nil_link"/>
     <child link="LARM_LINK6"/>
@@ -16,5 +16,5 @@
   </joint>
   <joint name="RHAND_DUMMY" type="revolute">
-    <origin xyz="0.30 0.30 0.40" rpy="3.14159 -1.5708 0"/>
+    <origin xyz="0.23 0.20 0.20" rpy="3.14159 -1.5708 0"/>
     <parent link="nil_link"/>
     <child link="RARM_LINK6"/>

File: hrpsys_gazebo_tutorials/environment_models/small_box/model3.urdf (robot description, URDF)
Before this commit: robot small_box, 15 links, 14 joints
Links:
- link nil_link3: geometry collision box size=0.20 0.315 0.61; visual box size=0.20 0.315 0.61
Joints:
- joint LHAND_DUMMY: origin xyz=0.30 -0.30 0.40 rpy=3.14159 -1.5708 0 -> xyz=0.23 -0.20 0.20 rpy=3.14159 -1.5708 0
- joint RHAND_DUMMY: origin xyz=0.30 0.30 0.40 rpy=3.14159 -1.5708 0 -> xyz=0.23 0.20 0.20 rpy=3.14159 -1.5708 0

File: hrpsys_gazebo_tutorials/environment_models/small_box/model3.urdf.xacro (robot description, xacro)
@@ -8,5 +8,5 @@
   </xacro:include>
   <joint name="LHAND_DUMMY" type="revolute">
-    <origin xyz="0.30 -0.30 0.40" rpy="3.14159 -1.5708 0"/>
+    <origin xyz="0.23 -0.20 0.20" rpy="3.14159 -1.5708 0"/>
     <parent link="nil_link"/>
     <child link="LARM_LINK6"/>
@@ -16,5 +16,5 @@
   </joint>
   <joint name="RHAND_DUMMY" type="revolute">
-    <origin xyz="0.30 0.30 0.40" rpy="3.14159 -1.5708 0"/>
+    <origin xyz="0.23 0.20 0.20" rpy="3.14159 -1.5708 0"/>
     <parent link="nil_link"/>
     <child link="RARM_LINK6"/>

File: hrpsys_gazebo_tutorials/environment_models/small_box/model4.urdf (robot description, URDF)
Before this commit: robot small_box, 15 links, 14 joints
Links:
- link nil_link4: geometry collision box size=0.20 0.315 0.61; visual box size=0.20 0.315 0.61
Joints:
- joint LHAND_DUMMY: origin xyz=0.30 -0.30 0.40 rpy=3.14159 -1.5708 0 -> xyz=0.23 -0.20 0.20 rpy=3.14159 -1.5708 0
- joint RHAND_DUMMY: origin xyz=0.30 0.30 0.40 rpy=3.14159 -1.5708 0 -> xyz=0.23 0.20 0.20 rpy=3.14159 -1.5708 0

File: hrpsys_gazebo_tutorials/environment_models/small_box/model4.urdf.xacro (robot description, xacro)
@@ -8,5 +8,5 @@
   </xacro:include>
   <joint name="LHAND_DUMMY" type="revolute">
-    <origin xyz="0.30 -0.30 0.40" rpy="3.14159 -1.5708 0"/>
+    <origin xyz="0.23 -0.20 0.20" rpy="3.14159 -1.5708 0"/>
     <parent link="nil_link"/>
     <child link="LARM_LINK6"/>
@@ -16,5 +16,5 @@
   </joint>
   <joint name="RHAND_DUMMY" type="revolute">
-    <origin xyz="0.30 0.30 0.40" rpy="3.14159 -1.5708 0"/>
+    <origin xyz="0.23 0.20 0.20" rpy="3.14159 -1.5708 0"/>
     <parent link="nil_link"/>
     <child link="RARM_LINK6"/>

File: hrpsys_gazebo_tutorials/environment_models/small_box/model5.urdf (robot description, URDF)
Before this commit: robot small_box, 15 links, 14 joints
Links:
- link nil_link5: geometry collision box size=0.20 0.315 0.61; visual box size=0.20 0.315 0.61
Joints:
- joint LHAND_DUMMY: origin xyz=0.30 -0.30 0.40 rpy=3.14159 -1.5708 0 -> xyz=0.23 -0.20 0.20 rpy=3.14159 -1.5708 0
- joint RHAND_DUMMY: origin xyz=0.30 0.30 0.40 rpy=3.14159 -1.5708 0 -> xyz=0.23 0.20 0.20 rpy=3.14159 -1.5708 0

File: hrpsys_gazebo_tutorials/environment_models/small_box/model5.urdf.xacro (robot description, xacro)
@@ -8,5 +8,5 @@
   </xacro:include>
   <joint name="LHAND_DUMMY" type="revolute">
-    <origin xyz="0.30 -0.30 0.40" rpy="3.14159 -1.5708 0"/>
+    <origin xyz="0.23 -0.20 0.20" rpy="3.14159 -1.5708 0"/>
     <parent link="nil_link"/>
     <child link="LARM_LINK6"/>
@@ -16,5 +16,5 @@
   </joint>
   <joint name="RHAND_DUMMY" type="revolute">
-    <origin xyz="0.30 0.30 0.40" rpy="3.14159 -1.5708 0"/>
+    <origin xyz="0.23 0.20 0.20" rpy="3.14159 -1.5708 0"/>
     <parent link="nil_link"/>
     <child link="RARM_LINK6"/>

File: hrpsys_gazebo_tutorials/environment_models/small_box/model6.urdf (robot description, URDF)
Before this commit: robot small_box, 15 links, 14 joints
Links:
- link nil_link6: geometry collision box size=0.20 0.315 0.61; visual box size=0.20 0.315 0.61
Joints:
- joint LHAND_DUMMY: origin xyz=0.30 -0.30 0.40 rpy=3.14159 -1.5708 0 -> xyz=0.23 -0.20 0.20 rpy=3.14159 -1.5708 0
- joint RHAND_DUMMY: origin xyz=0.30 0.30 0.40 rpy=3.14159 -1.5708 0 -> xyz=0.23 0.20 0.20 rpy=3.14159 -1.5708 0

File: hrpsys_gazebo_tutorials/environment_models/small_box/model6.urdf.xacro (robot description, xacro)
@@ -8,5 +8,5 @@
   </xacro:include>
   <joint name="LHAND_DUMMY" type="revolute">
-    <origin xyz="0.30 -0.30 0.40" rpy="3.14159 -1.5708 0"/>
+    <origin xyz="0.23 -0.20 0.20" rpy="3.14159 -1.5708 0"/>
     <parent link="nil_link"/>
     <child link="LARM_LINK6"/>
@@ -16,5 +16,5 @@
   </joint>
   <joint name="RHAND_DUMMY" type="revolute">
-    <origin xyz="0.30 0.30 0.40" rpy="3.14159 -1.5708 0"/>
+    <origin xyz="0.23 0.20 0.20" rpy="3.14159 -1.5708 0"/>
     <parent link="nil_link"/>
     <child link="RARM_LINK6"/>

File: hrpsys_gazebo_tutorials/environment_models/small_box/small_box1.urdf (robot description, URDF)
Before this commit: robot small_box-robot, 1 links, 0 joints
Links:
- link nil_link: geometry collision box size=0.20 0.315 0.61; visual box size=0.20 0.315 0.61

File: hrpsys_gazebo_tutorials/environment_models/small_box/small_box2.urdf (robot description, URDF)
Before this commit: robot small_box-robot, 1 links, 0 joints
Links:
- link nil_link: geometry collision box size=0.20 0.315 0.61; visual box size=0.20 0.315 0.61

File: hrpsys_gazebo_tutorials/environment_models/small_box/small_box3.urdf (robot description, URDF)
Before this commit: robot small_box-robot, 1 links, 0 joints
Links:
- link nil_link: geometry collision box size=0.20 0.315 0.61; visual box size=0.20 0.315 0.61

File: hrpsys_gazebo_tutorials/environment_models/small_box/small_box4.urdf (robot description, URDF)
Before this commit: robot small_box-robot, 1 links, 0 joints
Links:
- link nil_link: geometry collision box size=0.20 0.315 0.61; visual box size=0.20 0.315 0.61

File: hrpsys_gazebo_tutorials/environment_models/small_box/small_box5.urdf (robot description, URDF)
Before this commit: robot small_box-robot, 1 links, 0 joints
Links:
- link nil_link: geometry collision box size=0.20 0.315 0.61; visual box size=0.20 0.315 0.61

File: hrpsys_gazebo_tutorials/environment_models/small_box/small_box6.urdf (robot description, URDF)
Before this commit: robot small_box-robot, 1 links, 0 joints
Links:
- link nil_link: geometry collision box size=0.20 0.315 0.61; visual box size=0.20 0.315 0.61
